File: Hardware/iot_weatherstation_full_vcut.kicad_pcb (KiCad board)
At the start: 2 copper layers, 181 x 122.3 mm, 50 parts, among them IC1 ESP32-S3-WROOM-1-N8, IC2 VCNL4040M3OE, J1 USB-C_PD, J10 SolderJumper, J11 SolderJumper, J2 TTL, J3 SolderJumper, J4 SolderJumper, J6 JST-SH1.0-4P, J7 SolderJumper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

Commit message: Update gerber files
Routing:
- net GND: track 90.8 -> 59.6 mm
- net /BME688/SDA: track 238.9 -> 207.8 mm
- net +3V3: track 402.6 -> 371.5 mm
- net /BME688/SCL: track 234.5 -> 203.5 mm
Other:
- outline, holes or cut-outs redrawn
Changed lines of the file:
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@@
 		(end 310.3118 120.0404)
 		(stroke
-			(width 0.1)
+			(width 0.05)
 			(type default)
 		)
-		(layer "User.1")
+		(layer "Edge.Cuts")
 	)
 	(gr_line
-		(start 310.3118 120.0404)
-		(end 313.9948 120.0404)
+		(start 129.3114 120.0404)
+		(end 310.3118 120.0404)
 		(stroke
 			(width 0.1)
@@
 	)
 	(gr_line
-		(start 129.3114 120.0404)
-		(end 125.857 120.0404)
+		(start 310.3118 120.0404)
+		(end 313.9948 120.0404)
 		(stroke
 			(width 0.1)
@@
 	)
 	(gr_line
-		(start 313.867807 231.8512)
-		(end 123.720164 231.8512)
+		(start 129.3114 120.0404)
+		(end 125.857 120.0404)
 		(stroke
 			(width 0.1)
 			(type default)
 		)
-		(layer "User.9")
+		(layer "User.1")
 	)
 	(gr_text "5V"
@@
 	)
 	(segment
-		(start 139.5 134.5406)
-		(end 139.0028 135.0378)
-		(width 0.2)
-		(layer "B.Cu")
-		(net 1)
-	)
-	(segment
 		(start 137.9322 162.7248)
 		(end 137.9322 161.1884)
@@
 	)
 	(segment
-		(start 141.974381 113.78754)
-		(end 139.85686 113.78754)
-		(width 0.2)
-		(layer "B.Cu")
-		(net 1)
-	)
-	(segment
-		(start 139.85686 113.78754)
-		(end 139.5 114.1444)
-		(width 0.2)
-		(layer "B.Cu")
-		(net 1)
-	)
-	(segment
 		(start 307.5344 208.28)
 		(end 307.5344 199.9234)
@@
 	)
 	(segment
-		(start 139.0028 135.0378)
-		(end 131.507 135.0378)
-		(width 0.2)
-		(layer "B.Cu")
-		(net 1)
-	)
-	(segment
-		(start 139.5 114.1444)
-		(end 139.5 134.5406)
-		(width 0.2)
-		(layer "B.Cu")
-		(net 1)
-	)
-	(segment
 		(start 135.3444 131.699)
 		(end 135.3444 131.5554)
@@
 	)
 	(segment
-		(start 139.337 136.0498)
-		(end 131.507 136.0498)
-		(width 0.2)
-		(layer "B.Cu")
-		(net 2)
-	)
-	(segment
 		(start 139.4822 163.4738)
 		(end 139.4822 162.7248)
@@
 	)
 	(segment
-		(start 140.318798 114.798802)
-		(end 139.827 115.2906)
-		(width 0.2)
-		(layer "B.Cu")
-		(net 2)
-	)
-	(segment
 		(start 147.077 185.407)
 		(end 147.077 186.0298)
@@
 	)
 	(segment
-		(start 139.827 115.2906)
-		(end 139.827 135.5598)
-		(width 0.2)
-		(layer "B.Cu")
-		(net 2)
-	)
-	(segment
 		(start 150.4442 212.0138)
 		(end 149.365 212.0138)
@@
 	)
 	(segment
-		(start 141.926097 114.798802)
-		(end 140.318798 114.798802)
-		(width 0.2)
-		(layer "B.Cu")
-		(net 2)
-	)
-	(segment
 		(start 269.674383 110.70314)
 		(end 268.150383 110.70314)
@@
 	)
 	(segment
-		(start 139.827 135.5598)
-		(end 139.337 136.0498)
-		(width 0.2)
-		(layer "B.Cu")
-		(net 2)
-	)
-	(segment
 		(start 162.8712 163.1632)
 		(end 162.4132 163.6212)
@@
 	)
 	(segment
-		(start 141.907643 111.76)
-		(end 139.2936 111.76)
-		(width 0.2)
-		(layer "B.Cu")
-		(net 31)
-	)
-	(segment
 		(start 150.6452 183.9084)
 		(end 150.0996 184.454)
@@
 	)
 	(segment
-		(start 139.2936 111.76)
-		(end 138.846 112.2076)
-		(width 0.2)
-		(layer "B.Cu")
-		(net 31)
-	)
-	(segment
 		(start 221.541381 110.887938)
 		(end 221.558383 110.90494)
@@
 	)
 	(segment
-		(start 138.846 132.3498)
-		(end 138.146 133.0498)
-		(width 0.2)
-		(layer "B.Cu")
-		(net 31)
-	)
-	(segment
-		(start 138.146 133.0498)
-		(end 131.507 133.0498)
-		(width 0.2)
-		(layer "B.Cu")
-		(net 31)
-	)
-	(segment
-		(start 138.846 112.2076)
-		(end 138.846 132.3498)
-		(width 0.2)
-		(layer "B.Cu")
-		(net 31)
-	)
-	(segment
-		(start 141.940983 111.79334)
-		(end 141.907643 111.76)
-		(width 0.2)
-		(layer "B.Cu")
-		(net 31)
-	)
-	(segment
 		(start 150.0996 184.454)
 		(end 150.0996 185.407)
@@
 	)
 	(segment
-		(start 138.5938 134.0498)
-		(end 131.507 134.0498)
-		(width 0.2)
-		(layer "B.Cu")
-		(net 71)
-	)
-	(segment
 		(start 171.909781 112.78874)
 		(end 173.334983 112.78874)
@@
 	)
 	(segment
-		(start 139.173 113.2014)
-		(end 139.173 133.4706)
-		(width 0.2)
-		(layer "B.Cu")
-		(net 71)
-	)
-	(segment
-		(start 141.9352 112.79334)
-		(end 139.58106 112.79334)
-		(width 0.2)
-		(layer "B.Cu")
-		(net 71)
-	)
-	(segment
-		(start 139.173 133.4706)
-		(end 138.5938 134.0498)
-		(width 0.2)
-		(layer "B.Cu")
-		(net 71)
-	)
-	(segment
 		(start 148.727 185.407)
 		(end 148.727 186.1158)
@@
 		(width 0.2)
 		(layer "B.Cu")
-		(net 71)
-	)
-	(segment
-		(start 139.58106 112.79334)
-		(end 139.173 113.2014)
-		(width 0.2)
-		(layer "B.Cu")

Commit message: Swapped SCL und SDA for LTR (fucked up)
Connections:
- U3 pad 4: /BME688/SDA -> /BME688/SCL
- U3 pad 6: /BME688/SCL -> /BME688/SDA
Routing:
- net /BME688/SDA: track 207.8 -> 205.3 mm
- net /BME688/SCL: track 203.5 -> 205.0 mm
Changed lines of the file:
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@@
 			(size 0.3 0.65)
 			(layers "B.Cu" "B.Paste" "B.Mask")
-			(net 71 "/BME688/SDA")
+			(net 31 "/BME688/SCL")
 			(pinfunction "SCL")
 			(pintype "bidirectional")
@@
 			(size 0.3 0.65)
 			(layers "B.Cu" "B.Paste" "B.Mask")
-			(net 31 "/BME688/SCL")
+			(net 71 "/BME688/SDA")
 			(pinfunction "SDA")
 			(pintype "bidirectional")
@@
 	)
 	(segment
+		(start 262.48114 110.03034)
+		(end 262.6868 110.236)
+		(width 0.2)
+		(layer "F.Cu")
+		(net 31)
+	)
+	(segment
 		(start 143.283981 111.98614)
 		(end 143.283981 112.62114)
@@
 	(segment
 		(start 221.541381 110.03034)
-		(end 263.197381 110.03034)
+		(end 262.48114 110.03034)
 		(width 0.2)
 		(layer "F.Cu")
@@
 	)
 	(segment
-		(start 138.5496 133.0378)
-		(end 138.8872 133.3754)
+		(start 262.6868 112.3696)
+		(end 262.96374 112.64654)
 		(width 0.2)
 		(layer "F.Cu")
@@
 	)
 	(segment
-		(start 149.7362 180.8766)
-		(end 150.114 181.2544)
+		(start 262.6868 110.236)
+		(end 262.6868 112.3696)
 		(width 0.2)
 		(layer "F.Cu")
@@
 	)
 	(segment
-		(start 263.197381 110.03034)
-		(end 263.425981 110.25894)
+		(start 138.5496 133.0378)
+		(end 138.8872 133.3754)
+		(width 0.2)
+		(layer "F.Cu")
+		(net 31)
+	)
+	(segment
+		(start 149.7362 180.8766)
+		(end 150.114 181.2544)
 		(width 0.2)
 		(layer "F.Cu")
@@
 	)
 	(segment
-		(start 220.941381 110.63034)
-		(end 221.541381 110.03034)
+		(start 262.96374 112.64654)
+		(end 263.425981 112.64654)
 		(width 0.2)
 		(layer "F.Cu")
@@
 	)
 	(segment
-		(start 263.425981 110.25894)
-		(end 263.425981 111.35114)
+		(start 220.941381 110.63034)
+		(end 221.541381 110.03034)
 		(width 0.2)
 		(layer "F.Cu")
@@
 	)
 	(segment
+		(start 263.806981 112.64654)
+		(end 263.425981 112.64654)
+		(width 0.2)
+		(layer "F.Cu")
+		(net 31)
+	)
+	(segment
 		(start 143.487181 112.82434)
 		(end 170.436581 112.82434)
@@
 	)
 	(via
-		(at 263.425981 111.35114)
+		(at 131.507 133.0498)
 		(size 0.6)
 		(drill 0.3)
@@
 	)
 	(via
-		(at 131.507 133.0498)
+		(at 141.940983 111.79334)
 		(size 0.6)
 		(drill 0.3)
@@
 	)
 	(via
-		(at 141.940983 111.79334)
+		(at 263.425981 112.64654)
 		(size 0.6)
 		(drill 0.3)
@@
 	)
 	(segment
-		(start 264.171983 111.35114)
-		(end 264.182183 111.36134)
+		(start 173.311983 113.61174)
+		(end 173.337383 113.58634)
 		(width 0.2)
 		(layer "B.Cu")
@@
 	)
 	(segment
-		(start 173.311983 113.61174)
-		(end 173.337383 113.58634)
+		(start 264.167383 112.64654)
+		(end 264.182183 112.66134)
 		(width 0.2)
 		(layer "B.Cu")
@@
 	)
 	(segment
-		(start 150.0996 184.454)
-		(end 150.0996 185.407)
+		(start 263.425981 112.64654)
+		(end 264.167383 112.64654)
 		(width 0.2)
 		(layer "B.Cu")
@@
 	)
 	(segment
-		(start 263.425981 111.35114)
-		(end 264.171983 111.35114)
+		(start 150.0996 184.454)
+		(end 150.0996 185.407)
 		(width 0.2)
 		(layer "B.Cu")
@@
 	(segment
 		(start 221.292852 109.43034)
-		(end 263.841981 109.43034)
+		(end 263.15114 109.43034)
 		(width 0.2)
 		(layer "F.Cu")
@@
 	)
 	(segment
-		(start 220.474581 110.03034)
-		(end 220.692852 110.03034)
+		(start 148.7424 186.1312)
+		(end 148.7424 181.6608)
 		(width 0.2)
 		(layer "F.Cu")
@@
 	)
 	(segment
-		(start 148.7424 186.1312)
-		(end 148.7424 181.6608)
+		(start 263.425981 109.705181)
+		(end 263.425981 111.35114)
+		(width 0.2)
+		(layer "F.Cu")
+		(net 71)
+	)
+	(segment
+		(start 263.15114 109.43034)
+		(end 263.425981 109.705181)
+		(width 0.2)
+		(layer "F.Cu")
+		(net 71)
+	)
+	(segment
+		(start 220.692852 110.03034)
+		(end 221.292852 109.43034)
 		(width 0.2)
 		(layer "F.Cu")
@@
 	)
 	(segment
-		(start 263.841981 109.43034)
-		(end 264.025981 109.61434)
-		(width 0.2)
-		(layer "F.Cu")
-		(net 71)
-	)
-	(segment
 		(start 140.839981 112.79334)
 		(end 140.591581 112.54494)
@@
 	)
 	(segment
-		(start 218.848981 110.03034)
-		(end 220.474581 110.03034)
+		(start 220.474581 110.03034)
+		(end 220.692852 110.03034)
 		(width 0.2)
 		(layer "F.Cu")
@@
 	)
 	(segment
-		(start 141.320352 181.2036)
-		(end 139.954 179.837248)
+		(start 218.848981 110.03034)
+		(end 220.474581 110.03034)
 		(width 0.2)
 		(layer "F.Cu")
@@
 	)
 	(segment
-		(start 264.025981 109.61434)
-		(end 264.025981 112.42754)
+		(start 141.320352 181.2036)
+		(end 139.954 179.837248)
 		(width 0.2)
 		(layer "F.Cu")
@@
 	)
 	(segment
-		(start 264.025981 112.42754)
-		(end 263.806981 112.64654)
-		(width 0.2)
-		(layer "F.Cu")
-		(net 71)
-	)
-	(segment
 		(start 143.820581 112.49734)
 		(end 170.668381 112.49734)
@@
 	)
 	(segment
-		(start 263.806981 112.64654)
-		(end 263.425981 112.64654)
-		(width 0.2)
-		(layer "F.Cu")
-		(net 71)
-	)
-	(segment
 		(start 138.0002 134.0378)
 		(end 131.507 134.0378)
@@
 		(net 71)
 	)
-	(segment
-		(start 220.692852 110.03034)
-		(end 221.292852 109.43034)
-		(width 0.2)
-		(layer "F.Cu")
-		(net 71)
-	)
 	(via
 		(at 141.9352 112.79334)
@@
 	)
 	(via
-		(at 220.474581 110.03034)
+		(at 263.425981 111.35114)
 		(size 0.6)
 		(drill 0.3)
@@
 	)
 	(via
-		(at 131.507 134.0498)
+		(at 220.474581 110.03034)
 		(size 0.6)
 		(drill 0.3)
@@
 	)
 	(via
-		(at 148.7424 186.1312)
+		(at 131.507 134.0498)
 		(size 0.6)
 		(drill 0.3)
@@
 	)
 	(via
-		(at 171.909781 112.78874)
+		(at 148.7424 186.1312)
 		(size 0.6)
 		(drill 0.3)
@@
 	)
 	(via
-		(at 263.425981 112.64654)
+		(at 171.909781 112.78874)
 		(size 0.6)
 		(drill 0.3)
@@
 	)
 	(segment
-		(start 264.167383 112.64654)
-		(end 264.182183 112.66134)
+		(start 264.171983 111.35114)
+		(end 264.182183 111.36134)
 		(width 0.2)
 		(layer "B.Cu")
@@
 	)
 	(segment
-		(start 263.425981 112.64654)
-		(end 264.167383 112.64654)
-		(width 0.2)
-		(layer "B.Cu")
-		(net 71)
-	)
-	(segment
 		(start 173.334983 112.78874)
 		(end 173.337383 112.78634)
@@
 		(width 0.2)
 		(layer "B.Cu")
+		(net 71)
+	)
+	(segment
+		(start 263.425981 111.35114)
+		(end 264.171983 111.35114)
+		(width 0.2)
+		(layer "B.Cu")
